File: hw/canfd-usb-nucleo-expb/canfd-usb-nucleo-expb.sch (KiCad schematic (older format))
At the start: 58 parts, among them CN1 POWER, CN2 CONN, J1 USB_C_Receptacle_USB2.0, J2 Conn_01x10, J3 Conn_01x10, J4 Conn_01x10, SW1 SW_Push_Dual_x2, SW2 SW_Push_Dual_x2, SW3 SW_Push_Dual_x2, U1 USBLC6-2SC6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

Commit message: HW: First version of PCB layout
First version of PCB layout is ready for review.
Changed the assignments of pins for switches and status LEDs
to ease the routing of traces.
PCB's bottom layer is GND plane, most of the traces are placed
on top layer. Ground planes are connected with via stitching on
full area of the PCB.
There are no high speed signals on this PCB that might be of a concern
while routing so general rules of keeping the traces short and diff pairs
of the same lenghts are used.

Signed-off-by: AlexeyZ <silkt207@gmail.com>
Parts:
- added unit 6 of CN1
- CN1: value POWER -> Conn_02x19_Odd_Even
Connections:
- net LED1: now also CN2.1 (Pin_1)
- net LED2: now also CN1.21 (PB7)
- net LED3: now also CN1.30 (PA1)
- net LED4: now also CN1.34 (PB0); no longer CN2.1 (Pin_1)
- net RX2: now also CN2.23 (Pin_30); no longer CN2.3 (rx3)
- net RX3: now also CN2.3 (rx3); no longer CN2.23 (Pin_30)
- net STANDBY_1: now also R4.2; no longer R2.2
- net STANDBY_3: now also R2.2; no longer R4.2
- net SW1: now also CN1.32 (PA4)
- net SW2: now also CN1.28 (PA0)
- net SW3: now also CN1.4 (PD2)
- net TX2: now also CN2.27 (Pin_30); no longer CN2.5 (tx3)
- net TX3: now also CN2.5 (tx3); no longer CN2.27 (Pin_30)
Changed lines of the file:
@@
 Wire Wire Line
 	5250 2050 5500 2050
+Text GLabel 1350 2900 2    50   Output ~ 0
+TX3
+Text GLabel 1350 2300 2    50   Input ~ 0
+RX1
 Text GLabel 1350 2400 2    50   Output ~ 0
 TX1
 Text GLabel 1350 2550 2    50   Input ~ 0
-RX3
+RX2
 Text GLabel 1350 2650 2    50   Output ~ 0
-TX3
-Text GLabel 1350 2800 2    50   Input ~ 0
-RX2
-Text GLabel 1350 2900 2    50   Output ~ 0
 TX2
 Text GLabel 1350 3150 2    50   BiDi ~ 0
@@
 P 900 1600
 F 0 "CN1" H 979 1915 50  0000 C CNN
-F 1 "POWER" H 979 1824 50  0000 C CNN
+F 1 "Conn_02x19_Odd_Even" H 979 1824 50  0000 C CNN
 F 2 "Pin_Headers:Pin_Header_Straight_2x19_Pitch2.54mm" H 400 1150 50  0001 C CNN
 F 3 "" H 400 1150 50  0001 C CNN
@@
 	1    0    0    -1
 $EndComp
-Text GLabel 1350 2300 2    50   Input ~ 0
-RX1
+Text GLabel 1350 2800 2    50   Input ~ 0
+RX3
 Text GLabel 3350 1950 2    50   Output ~ 0
 SW2
@@
 U 5 1 5E62EF55
 P 1050 4550
-F 0 "CN2" H 1050 5550 50  0000 C CNN
+F 0 "CN2" H 1100 4950 50  0000 C CNN
 F 1 "CONN" H 1132 5576 50  0001 C CNN
 F 2 "Pin_Headers:Pin_Header_Straight_2x19_Pitch2.54mm" H 2100 4850 50  0001 C CNN
@@
 	1    0    0    -1
 $EndComp
-Text GLabel 1350 3650 2    50   Input ~ 0
+Text GLabel 1400 3900 2    50   Input ~ 0
 SW1
-Text GLabel 1350 3750 2    50   Input ~ 0
+Text GLabel 1400 3700 2    50   Input ~ 0
 SW2
-Text GLabel 1350 3850 2    50   Input ~ 0
+Text GLabel 1400 3500 2    50   Input ~ 0
 SW3
-Text GLabel 1350 3950 2    50   Output ~ 0
+Text GLabel 1350 4250 2    50   Output ~ 0
 LED1
-Text GLabel 1350 4050 2    50   Output ~ 0
+Text GLabel 1400 3600 2    50   Output ~ 0
 LED2
-Text GLabel 1350 4150 2    50   Output ~ 0
+Text GLabel 1400 3800 2    50   Output ~ 0
 LED3
-Text GLabel 1350 4250 2    50   Output ~ 0
+Text GLabel 1400 4000 2    50   Output ~ 0
 LED4
 Text GLabel 2950 3600 0    50   Input ~ 0
@@
 	5250 2200 5500 2200
 Text GLabel 1950 4550 2    50   Output ~ 0
-STANDBY_3
+STANDBY_1
 Text GLabel 1950 4450 2    50   Output ~ 0
 STANDBY_2
 Text GLabel 1950 4350 2    50   Output ~ 0
-STANDBY_1
+STANDBY_3
 Wire Wire Line
 	7100 3650 7350 3650
@@
 Wire Wire Line
 	2850 5900 3150 5900
+$Comp
+L canfd-usb-nucleo:Conn_02x19_Odd_Even CN1
+U 6 1 5E95CC46
+P 1100 3750
+F 0 "CN1" H 1207 4216 50  0000 C CNN
+F 1 "Conn_02x19_Odd_Even" H 1207 4125 50  0000 C CNN
+F 2 "Pin_Headers:Pin_Header_Straight_2x19_Pitch2.54mm" H 2150 4050 50  0001 C CNN
+F 3 "" H 2150 4050 50  0001 C CNN
+	6    1100 3750
+	1    0    0    -1
+$EndComp
 $EndSCHEMATC
